Commit message: commit 3 - rviz

File: urdf/robot.urdf (robot description, URDF)
Before this commit: robot my-robot, 5 links, 4 joints
Joints:
- joint base_joint: origin xyz=0 0 0.5 rpy=0 0 0 -> xyz=0 0 0.31 rpy=0 0 0

Commit message: commit 4

File: urdf/robot.urdf (robot description, URDF)
Before this commit: robot my-robot, 5 links, 4 joints
Links:
- added link lidar_link
Joints:
- added joint lidar_joint: type fixed, parent body, child lidar_link, origin xyz=-0.148 0.37 0.5 rpy=0 0 0

Commit message: commit 5 - gazebo

File: urdf/robot.urdf (robot description, URDF)
Before this commit: robot my-robot, 6 links, 5 joints
Links:
- link spherical_wheel: mass 2.48241 -> 2.48
- link standard_wheel: mass 0.465267 -> 0.465
- link standard_wheel_2: mass 0.465267 -> 0.465
Joints:
- removed joint joint_left_wheel
- removed joint joint_right_wheel
- added joint front_left_wheel_joint: type continuous, parent body, child standard_wheel, origin xyz=0.0788842 0.476898 -0.250217 rpy=-1.5708 -0 1.5708, axis 0 0 1, limit effort=20 velocity=20
- added joint front_right_wheel_joint: type continuous, parent body, child standard_wheel_2, origin xyz=-0.381116 0.476898 -0.250217 rpy=1.5708 -0 1.5708, axis 0 0 -1, limit effort=20 velocity=20
- joint joint_spherical_wheel: axis 0 0 1 -> (none); limit effort=10 velocity=10 -> (none); origin xyz=-0.151116 0.201898 -0.265217 rpy=0 -0 2.42861e-16 -> xyz=-0.151116 0.201898 -0.265217 rpy=0 0 0
- joint lidar_joint: origin xyz=-0.148 0.37 0.5 rpy=0 0 0 -> xyz=-0.148 0.4 0.5 rpy=0 0 0

Commit message: commit 18 - change lidar position

File: urdf/robot.urdf (robot description, URDF)
Before this commit: robot my-robot, 6 links, 5 joints
Joints:
- joint lidar_joint: origin xyz=-0.148 0.4 0.5 rpy=0 0 0 -> xyz=-0.15 0.4 0.2 rpy=0 0 0

Commit message: commit 19 - fix robot orientation

File: urdf/robot.urdf (robot description, URDF)
Before this commit: robot my-robot, 6 links, 5 joints
Links:
- removed link standard_wheel
- removed link standard_wheel_2
- added link left_wheel, mass 0.465267; collision mesh filename=package://hospital_robot/meshes/standard_wheel.stl; visual mesh filename=package://hospital_robot/meshes/standard_wheel.stl
- added link right_wheel, mass 0.465267; collision mesh filename=package://hospital_robot/meshes/standard_wheel.stl; visual mesh filename=package://hospital_robot/meshes/standard_wheel.stl
Joints:
- removed joint front_left_wheel_joint
- removed joint front_right_wheel_joint
- added joint left_wheel_joint: type continuous, parent body, child left_wheel, origin xyz=-0.23 -0.102937 0.0575 rpy=-1.5708 -0 -1.5708, axis 0 0 -1, limit effort=20 velocity=20
- added joint right_wheel_joint: type continuous, parent body, child right_wheel, origin xyz=0.23 -0.102937 0.0575 rpy=1.5708 -0 -1.5708, axis 0 0 1, limit effort=20 velocity=20
- joint joint_spherical_wheel: origin xyz=-0.151116 0.201898 -0.265217 rpy=0 0 0 -> xyz=2.52012e-17 0.172063 0.0425 rpy=0 -0 2.42861e-16
- joint lidar_joint: origin xyz=-0.15 0.4 0.2 rpy=0 0 0 -> xyz=0 0 0.2 rpy=0 0 0

Commit message: commit 20 - change lidar z value

File: urdf/robot.urdf (robot description, URDF)
Before this commit: robot my-robot, 6 links, 5 joints
Joints:
- joint lidar_joint: origin xyz=0 0 0.2 rpy=0 0 0 -> xyz=0 0 0.5 rpy=0 0 0
